File: Arduino_clone_4_layer.kicad_pcb (KiCad board)
At the start: 4 copper layers, 42 x 29 mm, 17 parts, among them J1 Serial, J2 Digital pins, J3 I2C, J4 ICSP, U1 24LC1025, U2 24LC1025, U3 DS1337S+, U4 ATMEGA328P-AU, Y1 32 MHz, Y2 16 MHz

Commit message: Added ground fill to 4-layer design
Routing:
- added copper zone on In2.Cu, net GNDPWR
